File: elecStack/Stack/MainBoard_v1.0.0/MainBoard_v1.0.0.kicad_sch (KiCad schematic)
At the start: 28 parts, among them J1 Conn_01x04_Socket, J2 Conn_01x06_Pin, J3 Conn_01x06_Pin, J4 Conn_01x20_Socket, J5 Conn_01x20_Socket, Q1 NMOS, Q2 NMOS, Q3 NMOS, Q4 NMOS, Q5 NMOS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

Commit message: Updated version 1
Connections:
- net TOGG4: no longer U3.7 (A6)
- new net TOGG5: U3.7 (A6)
Changed lines of the file:
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@@
 		)
 	)
-	(global_label "TOGG4"
+	(global_label "TOGG5"
 		(shape input)
 		(at 46.99 177.8 180)

Commit message: Make changes indicated in the schematic
Parts:
- removed J4, J5: Conn_01x20_Socket, symbol Connector:Conn_01x20_Socket
Connections:
- net 3V3: no longer U4.16 (VCC1)
- net 5V_LVL_SHFT_1: no longer U4.2 (1A)
- net 5V_LVL_SHFT_4: now also U3.14 (B6); no longer U3.13 (B7)
- net 5V_LVL_SHFT_5: now also U3.13 (B7); no longer U3.14 (B6)
- net 5V_buck: now also U4.16 (VCC1); no longer U4.8 (VCC2)
- net PWR_IN: now also U4.8 (VCC2)
- net TOGG4: now also U3.7 (A6); no longer U3.8 (A7)
- net TOGG5: now also U1.GP16, U3.8 (A7); no longer U3.7 (A6)
- net 5V_LVL_SHFT_6: now reaches U3.16 (B4)
- net 5V_LVL_SHFT_6: now also U4.2 (1A)
- net TOGG6: now reaches U3.5 (A4)
- net TOGG6: now also U1.GP15
Other:
- note added: "Make IMU connections over I2C"
