File: elecStack/Stack/MainBoard_v1.0.0/MainBoard_v1.0.0.kicad_sch (KiCad schematic)
At the start: 48 parts, among them J1 Conn_01x04_Socket, Q1 NMOS, Q2 NMOS, Q3 NMOS, Q4 NMOS, Q5 NMOS, Q6 NMOS, Q7 NMOS, Q8 PMOS, SW1 SW_Push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

Commit message: updated_11_march
Parts:
- added C2, C3, C4, C5: 0.1uF, Capacitor_SMD:C_1210_3225Metric_Pad1.33x2.70mm_HandSolder, symbol Device:C
- U3, U5: footprint Package_SO:TSSOP-20_4.4x6.5mm_P0.65mm -> Connector_PinHeader_2.54mm:PinHeader_1x10_P2.54mm_Vertical_1
Connections:
- net 3V3: now also C2.2, C5.1
- net 5V_buck: now also C3.1, C4.1
- net GND: now also C2.1, C3.2, C4.2, C5.2
