File: elecStack/Stack/MainBoard_v1.0.0/connectors.kicad_sch (KiCad schematic)
At the start: 9 parts, among them J10 Conn_01x02_Socket, J2 Conn_01x06_Pin, J3 Conn_01x06_Pin, J4 Conn_01x02_Socket, J5 Conn_01x02_Socket, J6 Conn_01x07_Pin, J8 Conn_01x02_Socket, J9 Conn_01x02_Socket, U6 L293D

Commit message: Routing done
Parts:
- added D10: ASMB-MTB0-0A3A2, LED_THT:LED_D5.0mm-4_RGB, symbol LED:ASMB-MTB0-0A3A2_CC
- added R14: 220, Resistor_SMD:R_0805_2012Metric_Pad1.20x1.40mm_HandSolder, symbol Device:R
- J5: footprint Connector_PinHeader_2.54mm:PinHeader_1x02_P2.54mm_Vertical -> Connector_Phoenix_MSTB:PhoenixContact_MSTBA_2,5_2-G_1x02_P5.00mm_Horizontal
Connections:
- net GP15 is gone; now on net GND: J6.7 (Pin_7)
- net GND: now also R14.2
- net GP3 renamed GP3_5V
- net GP4 renamed GP4_5V
- net GP5 renamed GP5_5V
- net GP6 renamed GP6_5V
- net GP7 renamed GP7_5V
- net GP9 renamed GP8_5V
- net INT: no longer names the net of J3.1 (Pin_1)
- net RXD_MD renamed RXD_MD_5V
- net TXD_MD renamed TXD_MD_5V
- new net: D10.1 (A), R14.1
- new net LED_PIN_1: D10.4 (RK)
- new net LED_PIN_2: D10.3 (GK)
- new net LED_PIN_3: D10.2 (BK)
- no-connect marks 9 -> 10
Other:
- moved on the sheet: J5, U6

Commit message: version 1.2.0 layout done
Parts:
- removed J10, J4, J8, J9: Conn_01x02_Socket, Connector_Phoenix_MSTB:PhoenixContact_MSTBA_2,5_2-G_1x02_P5.00mm_Horizontal, symbol Connector:Conn_01x02_Socket
- added J10, J7, J8, J9: Conn_01x03_Socket, Connector_JST:JST_EH_B3B-EH-A_1x03_P2.50mm_Vertical, symbol Connector:Conn_01x03_Socket
Connections:
- net GND: now also J10.3 (Pin_3), J7.3 (Pin_3), J8.3 (Pin_3), J9.3 (Pin_3)
- net RXD_MD_5V: now also J10.1 (Pin_1), J7.2 (Pin_2), J8.2 (Pin_2), J9.2 (Pin_2)
- net TXD_MD_5V: now also J10.2 (Pin_2), J7.1 (Pin_1), J8.1 (Pin_1), J9.1 (Pin_1)
