File: elecStack/Stack/MainBoard_v1.2.0/MainBoard_v1.2.0.kicad_pcb (KiCad board)
At the start: 2 copper layers, 126.5 x 101.5 mm, 62 parts, among them J1 Conn_01x04_Socket, J2 Conn_01x06_Pin, J3 Conn_01x06_Pin, J4 Conn_01x07_Socket, J5 Conn_01x07_Socket, J6 Conn_01x04_Socket, Q1 NMOS, SW1 SW_Push, SW2 SW_Wuerth_450301014042, U1 RASPBERRY_PI_PICO

Commit message: routing done
Parts:
- removed D1, D15, D16, D17, D18, D19, D8, D9: GREEN_LED, LED_SMD:LED_0805_2012Metric_Pad1.15x1.40mm_HandSolder
- removed J1: Conn_01x04_Socket, Connector_Phoenix_MSTB:PhoenixContact_MSTBA_2,5_4-G_1x04_P5.00mm_Horizontal
- removed J6: Conn_01x04_Socket, Connector_PinHeader_2.54mm:PinHeader_1x04_P2.54mm_Vertical
- removed R11, R17, R20, R21, R22, R24, R3, R6: 150, Resistor_SMD:R_0805_2012Metric_Pad1.20x1.40mm_HandSolder
- added BATTERY_CONN2: Conn_01x02_Socket, TerminalBlock_Phoenix:TerminalBlock_Phoenix_MKDS-1,5-2-5.08_1x02_P5.08mm_Horizontal, F.Cu at (59.8, 94.5)
- added BATTERY_CONN3: Conn_01x02_Socket, TerminalBlock_Phoenix:TerminalBlock_Phoenix_MKDS-1,5-2-5.08_1x02_P5.08mm_Horizontal, F.Cu at (60.0, 107.5)
- added J10: Conn_01x04_Socket, Connector_JST:JST_XH_B4B-XH-A_1x04_P2.50mm_Vertical, F.Cu at (58.0, 130.2)
- added J11: Conn_01x04_Socket, Connector_JST:JST_XH_B4B-XH-A_1x04_P2.50mm_Vertical, F.Cu at (72.4, 95.1)
- added J12: Conn_01x04_Socket, Connector_JST:JST_XH_B4B-XH-A_1x04_P2.50mm_Vertical, F.Cu at (146.5, 103.0)
- added J7: Conn_01x06_Socket, Connector_JST:JST_XH_B6B-XH-A_1x06_P2.50mm_Vertical, F.Cu at (97.0, 95.1)
- added J8: Conn_01x02_Pin, TerminalBlock_Phoenix:TerminalBlock_Phoenix_MKDS-1,5-2-5.08_1x02_P5.08mm_Horizontal, F.Cu at (136.0, 97.2)
- added J9: Conn_01x02_Pin, TerminalBlock_Phoenix:TerminalBlock_Phoenix_MKDS-1,5-2-5.08_1x02_P5.08mm_Horizontal, F.Cu at (139.0, 151.3)
- BATTERY_CONN1: footprint Connector_Phoenix_MSTB:PhoenixContact_MSTBA_2,5_2-G-5,08_1x02_P5.08mm_Horizontal -> TerminalBlock_Phoenix:TerminalBlock_Phoenix_MKDS-1,5-2-5.08_1x02_P5.08mm_Horizontal
- J4: value Conn_01x07_Socket -> Conn_01x06_Socket; footprint Connector_JST:JST_XH_B7B-XH-A_1x07_P2.50mm_Vertical -> Connector_JST:JST_XH_B6B-XH-A_1x06_P2.50mm_Vertical
- J5: value Conn_01x07_Socket -> Conn_01x04_Socket; footprint Connector_JST:JST_XH_B7B-XH-A_1x07_P2.50mm_Vertical -> Connector_JST:JST_XH_B4B-XH-A_1x04_P2.50mm_Vertical
- moved R31 61.4 mm to (138.3, 110.7), turned to 180 degrees
- moved J4 60.3 mm to (99.9, 155.5)
- moved R27 48.7 mm to (72.0, 105.5), turned to -90 degrees
- moved R33 47.7 mm to (137.2, 106.6)
- moved R13 41.8 mm to (132.7, 106.4), turned to 180 degrees
- moved R7 34.9 mm to (82.6, 104.2), turned to -90 degrees
- moved D4 34.2 mm to (82.4, 109.7), turned to 90 degrees
- moved R8 34.1 mm to (86.0, 104.2), turned to -90 degrees
- moved R9 33.3 mm to (89.4, 104.1), turned to -90 degrees
- moved D5 33.3 mm to (85.9, 109.6), turned to 90 degrees
- moved R10 32.8 mm to (92.7, 104.1), turned to -90 degrees
- moved D6 32.6 mm to (89.3, 109.7), turned to 90 degrees
- moved D7 32.0 mm to (92.5, 109.6), turned to 90 degrees
- moved R29 31.8 mm to (70.5, 109.5), turned to 180 degrees
- moved R23 29.6 mm to (64.7, 130.3), turned to 0 degrees
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Connections:
- J3 pad 5: 3V -> unconnected-(J3-Pin_5-Pad5)
- J4 pad 1: PWR_IN -> EN_3
- J4 pad 2: EN_1 -> EN_4
- J4 pad 3: IN_1_1 -> IN_1_3
- J4 pad 4: IN_2_1 -> IN_2_3
- J4 pad 5: IN_1_2 -> IN_1_4
- J4 pad 6: IN_2_2 -> IN_2_4
- J5 pad 1: PWR_IN -> ENC_A_1
- J5 pad 2: EN_3 -> ENC_B_1
- J5 pad 3: IN_1_3 -> 5V_buck
- J5 pad 4: IN_2_3 -> GND
- U1 pad GP16: EN_4 -> ENC_A_4_3.3
- U1 pad GP28_A2: V_measure -> unconnected-(U1-PadGP28_A2)
- U1 pad GP4: ENC_A_4_3.3 -> EN_3
- U1 pad GP5: EN_3 -> EN_4
Routing:
- net PWR_IN: track 0.00 -> 210.2 mm
- net 5V_buck: track 0.00 -> 192.9 mm, vias 0 -> 1
- net 3V3: track 0.00 -> 84.3 mm
- net 12_V_battery: track 0.00 -> 53.8 mm
- net IN_1_1: track 0.00 -> 49.1 mm, vias 0 -> 1
- net IN_1_3: track 0.00 -> 48.1 mm, vias 0 -> 1
- net IN_2_3: track 0.00 -> 47.7 mm, vias 0 -> 1
- net IN_1_4: track 0.00 -> 47.5 mm, vias 0 -> 1
- net IN_2_1: track 0.00 -> 47.5 mm, vias 0 -> 1
- net IN_1_2: track 0.00 -> 46.3 mm, vias 0 -> 1
- net Net-(JP1-A): track 0.00 -> 45.7 mm
- net IN_2_2: track 0.00 -> 45.6 mm, vias 0 -> 1
- net IN_2_4: track 0.00 -> 44.9 mm, vias 0 -> 1
- net RST: track 0.00 -> 39.3 mm
- net ENC_A_3_3.3: track 0.00 -> 38.0 mm, vias 0 -> 1
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Other:
- board size 126.5 x 101.5 mm -> 99.8 x 77.6 mm

Commit message: final_PCB
Parts:
- removed D10: ASMB-MTB0-0A3A2, LED_THT:LED_D5.0mm-4_RGB
- added BATTERY_CONN4: Conn_01x02_Socket, TerminalBlock_Phoenix:TerminalBlock_Phoenix_MKDS-1,5-2-5.08_1x02_P5.08mm_Horizontal, F.Cu at (72.9, 94.4)
- added J1: Conn_01x04_Socket, Connector_JST:JST_XH_B4B-XH-A_1x04_P2.50mm_Vertical, F.Cu at (144.9, 148.6)
- added J13: Conn_01x03_Socket, Connector_JST:JST_XH_B3B-XH-A_1x03_P2.50mm_Vertical, F.Cu at (104.1, 159.5)
- added J14: Conn_01x02_Socket, Connector_JST:JST_XH_B2B-XH-A_1x02_P2.50mm_Vertical, F.Cu at (144.6, 134.4)
- added J15: Conn_01x02_Pin, TerminalBlock_Phoenix:TerminalBlock_Phoenix_MKDS-1,5-2-5.08_1x02_P5.08mm_Horizontal, F.Cu at (139.3, 93.7)
- added J6: Conn_01x03_Socket, Connector_JST:JST_XH_B3B-XH-A_1x03_P2.50mm_Vertical, F.Cu at (95.8, 93.6)
- added REF**: MountingHole_3.2mm_M3, MountingHole:MountingHole_3.2mm_M3, F.Cu at (119.4, 122.0)
- added REF**: MountingHole_3.2mm_M3, MountingHole:MountingHole_3.2mm_M3, F.Cu at (129.4, 153.0)
- added REF**: MountingHole_3.2mm_M3, MountingHole:MountingHole_3.2mm_M3, F.Cu at (68.8, 117.8)
- J4, J7: value Conn_01x06_Socket -> Conn_01x03_Socket; footprint Connector_JST:JST_XH_B6B-XH-A_1x06_P2.50mm_Vertical -> Connector_JST:JST_XH_B3B-XH-A_1x03_P2.50mm_Vertical
- Q1: footprint Connector_Molex:Molex_SPOX_5267-03A_1x03_P2.50mm_Vertical -> Connector_Molex:IRF540N
- R1: value 220 -> 50k
- moved R1 68.5 mm to (74.8, 151.1), turned to 90 degrees
- moved J7 11.2 mm to (108.0, 93.5)
- moved J8 10.4 mm to (126.2, 93.8)
- moved J11 8.88 mm to (80.8, 92.5)
- moved C1 8.63 mm to (132.7, 102.6)
- moved J9 8.43 mm to (142.2, 159.1)
- moved J4 8.05 mm to (92.9, 159.5)
- moved R13 7.34 mm to (138.5, 101.9)
- moved J5 5.64 mm to (79.3, 159.4)
- moved SW1 5.25 mm to (120.7, 102.8), turned to 0 degrees
- moved BATTERY_CONN2 4.78 mm to (57.1, 98.5)
- moved J3 4.43 mm to (133.0, 143.6)
- moved JP1 4.00 mm to (143.9, 125.5)
- moved BATTERY_CONN3 3.87 mm to (57.3, 110.2)
- moved J2 3.43 mm to (120.3, 160.7)
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Connections:
- J2 pad 4: RST -> unconnected-(J2-Pin_4-Pad4)
- J3 pad 2: SDA -> 3V3
- J3 pad 3: SCL -> GND
- J3 pad 4: GND -> SDA
- J3 pad 5: unconnected-(J3-Pin_5-Pad5) -> SCL
- J3 pad 6: 3V3 -> RST
- J4 pad 2: EN_4 -> IN_1_3
- J4 pad 3: IN_1_3 -> IN_2_3
- J7 pad 1: EN_1 -> IN_1_2
- J7 pad 2: IN_1_1 -> IN_2_2
- J7 pad 3: IN_2_1 -> EN_2
- R1 pad 1: Net-(D10-A) -> Net-(Q1-G)
- U1 pad GP10: IN_2_4 -> EN_4
- U1 pad GP13: LED_PIN_1 -> GP13
- U1 pad GP14: LED_PIN_2 -> GP14
- U1 pad GP15: LED_PIN_3 -> GP15
- U1 pad GP5: EN_4 -> IN_1_3
- U1 pad GP6: IN_1_3 -> IN_2_3
- U1 pad GP7: IN_2_3 -> IN_1_4
- U1 pad GP8: IN_1_4 -> IN_2_4
- U1 pad VBUS: 5V_buck -> unconnected-(U1-PadVBUS)
- U1 pad VSYS: unconnected-(U1-PadVSYS) -> 5V_buck
Routing:
- net 5V_buck: track 192.9 -> 304.5 mm
- net PWR_IN: track 210.2 -> 309.8 mm
- net TOGG_ACT_2: track 0.00 -> 53.6 mm
- net TOGG_ACT_1: track 0.00 -> 50.0 mm
- net GP13: track 0.00 -> 34.5 mm
- net GP14: track 0.00 -> 28.3 mm
- net GP15: track 0.00 -> 24.9 mm
- net LED_PIN_1: track 24.1 -> 0.00 mm
- net GND_battery: track 10.9 -> 34.9 mm, vias 0 -> 1
- net LED_PIN_2: track 17.6 -> 0.00 mm
- net LED_PIN_3: track 14.5 -> 0.00 mm
- net RST: track 39.3 -> 29.3 mm
- net ENC_A_3: track 9.56 -> 17.1 mm
- net 3V3: track 84.3 -> 77.3 mm
- net IN_2_2: track 45.6 -> 51.8 mm
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Other:
- board size 99.8 x 77.6 mm -> 99.8 x 78.3 mm
- board text added: "TUE-05"
