File: elecStack/Stack/MainBoard_v1.2.0/MainBoard_v1.2.0.kicad_sch (KiCad schematic)
At the start: 62 parts, among them J1 Conn_01x04_Socket, J2 Conn_01x06_Pin, J3 Conn_01x06_Pin, J4 Conn_01x07_Socket, J5 Conn_01x07_Socket, J6 Conn_01x04_Socket, Q1 NMOS, SW1 SW_Push, SW2 SW_Wuerth_450301014042, U1 RASPBERRY_PI_PICO

Commit message: routing done
Parts:
- removed D1, D15, D16, D17, D18, D19, D8, D9: GREEN_LED, LED_SMD:LED_0805_2012Metric_Pad1.15x1.40mm_HandSolder, symbol Device:LED
- removed J1: Conn_01x04_Socket, Connector_Phoenix_MSTB:PhoenixContact_MSTBA_2,5_4-G_1x04_P5.00mm_Horizontal, symbol Connector:Conn_01x04_Socket
- removed J4, J5: Conn_01x07_Socket, Connector_JST:JST_XH_B7B-XH-A_1x07_P2.50mm_Vertical, symbol Connector:Conn_01x07_Socket
- removed J6: Conn_01x04_Socket, Connector_PinHeader_2.54mm:PinHeader_1x04_P2.54mm_Vertical, symbol Connector:Conn_01x04_Socket
- removed R11, R17, R20, R21, R22, R24, R3, R6: 150, Resistor_SMD:R_0805_2012Metric_Pad1.20x1.40mm_HandSolder, symbol Device:R
- added BATTERY_CONN2, BATTERY_CONN3: Conn_01x02_Socket, TerminalBlock_Phoenix:TerminalBlock_Phoenix_MKDS-1,5-2-5.08_1x02_P5.08mm_Horizontal, symbol Connector:Conn_01x02_Socket
- added J10, J11, J12, J5: Conn_01x04_Socket, Connector_JST:JST_XH_B4B-XH-A_1x04_P2.50mm_Vertical, symbol Connector:Conn_01x04_Socket
- added J4, J7: Conn_01x06_Socket, Connector_JST:JST_XH_B6B-XH-A_1x06_P2.50mm_Vertical, symbol Connector:Conn_01x06_Socket
- added J8, J9: Conn_01x02_Pin, TerminalBlock_Phoenix:TerminalBlock_Phoenix_MKDS-1,5-2-5.08_1x02_P5.08mm_Horizontal, symbol Connector:Conn_01x02_Pin
- BATTERY_CONN1: footprint Connector_Phoenix_MSTB:PhoenixContact_MSTBA_2,5_2-G-5,08_1x02_P5.08mm_Horizontal -> TerminalBlock_Phoenix:TerminalBlock_Phoenix_MKDS-1,5-2-5.08_1x02_P5.08mm_Horizontal
Connections:
- net 5V_buck: now also BATTERY_CONN2.1 (Pin_1), J10.3 (Pin_3), J11.3 (Pin_3), J12.3 (Pin_3), J5.3 (Pin_3)
- net ENC_A_1: now also J5.1 (Pin_1)
- net ENC_A_2: now also J10.1 (Pin_1)
- net ENC_A_3: now also J11.1 (Pin_1)
- net ENC_A_4: now also J12.4 (Pin_4)
- net ENC_A_4_3.3: now also U1.GP16; no longer U1.GP4
- net EN_1: now also J7.1 (Pin_1)
- net EN_2: now also J7.6 (Pin_6)
- net EN_3: now also U1.GP4, J4.1 (Pin_1); no longer U1.GP5
- net EN_4: now also U1.GP5, J4.2 (Pin_2); no longer U1.GP16
- net GND: now also BATTERY_CONN2.2 (Pin_2), BATTERY_CONN3.1 (Pin_1), J10.4 (Pin_4), J11.4 (Pin_4), J12.1 (Pin_1), J5.4 (Pin_4), J8.2 (Pin_2), J9.2 (Pin_2)
- net IN_1_1: now also J7.2 (Pin_2)
- net IN_1_2: now also J7.4 (Pin_4)
- net IN_1_3: now also J4.3 (Pin_3)
- net IN_1_4: now also J4.5 (Pin_5)
- net IN_2_1: now also J7.3 (Pin_3)
- net IN_2_2: now also J7.5 (Pin_5)
- net IN_2_3: now also J4.4 (Pin_4)
- net IN_2_4: now also J4.6 (Pin_6)
- net PWR_IN: now also BATTERY_CONN3.2 (Pin_2), J8.1 (Pin_1), J9.1 (Pin_1)
- net 3V: no longer names the net of J3.5 (Pin_5)
- net V_measure: no longer names the net of U1.GP28_A2
- new net ENC_B_1: J5.2 (Pin_2)
- new net ENC_B_2: J10.2 (Pin_2)
- new net ENC_B_3: J11.2 (Pin_2)
- new net ENC_B_4: J12.2 (Pin_2)
- no-connect marks 10 -> 12

Commit message: final_PCB
Parts:
- removed D10: ASMB-MTB0-0A3A2, LED_THT:LED_D5.0mm-4_RGB, symbol LED:ASMB-MTB0-0A3A2_CC
- removed J4, J7: Conn_01x06_Socket, Connector_JST:JST_XH_B6B-XH-A_1x06_P2.50mm_Vertical, symbol Connector:Conn_01x06_Socket
- added BATTERY_CONN4: Conn_01x02_Socket, TerminalBlock_Phoenix:TerminalBlock_Phoenix_MKDS-1,5-2-5.08_1x02_P5.08mm_Horizontal, symbol Connector:Conn_01x02_Socket
- added J1: Conn_01x04_Socket, Connector_JST:JST_XH_B4B-XH-A_1x04_P2.50mm_Vertical, symbol Connector:Conn_01x04_Socket
- added J13, J4, J6, J7: Conn_01x03_Socket, Connector_JST:JST_XH_B3B-XH-A_1x03_P2.50mm_Vertical, symbol Connector:Conn_01x03_Socket
- added J14: Conn_01x02_Socket, Connector_JST:JST_XH_B2B-XH-A_1x02_P2.50mm_Vertical, symbol Connector:Conn_01x02_Socket
- added J15: Conn_01x02_Pin, TerminalBlock_Phoenix:TerminalBlock_Phoenix_MKDS-1,5-2-5.08_1x02_P5.08mm_Horizontal, symbol Connector:Conn_01x02_Pin
- Q1: footprint Connector_Molex:Molex_SPOX_5267-03A_1x03_P2.50mm_Vertical -> Connector_Molex:IRF540N
- R1: value 220 -> 50k
Connections:
- net 3V3: now also J3.2 (Pin_2); no longer J3.6 (Pin_6)
- net 5V_buck: now also U1.VSYS, BATTERY_CONN4.1 (Pin_1); no longer U1.VBUS
- net EN_1: now also J6.1 (Pin_1)
- net EN_2: now also J7.3 (Pin_3)
- net EN_3: now also J4.1 (Pin_1)
- net EN_4: now also U1.GP10, J13.3 (Pin_3); no longer U1.GP5
- net GND: now also J3.3 (Pin_3), BATTERY_CONN4.2 (Pin_2), J1.4 (Pin_4), J15.2 (Pin_2); no longer J3.4 (Pin_4)
- net IN_1_1: now also J6.2 (Pin_2)
- net IN_1_2: now also J7.1 (Pin_1)
- net IN_1_3: now also U1.GP5, J4.2 (Pin_2); no longer U1.GP6
- net IN_1_4: now also U1.GP7, J13.1 (Pin_1); no longer U1.GP8
- net IN_2_1: now also J6.3 (Pin_3)
- net IN_2_2: now also J7.2 (Pin_2)
- net IN_2_3: now also U1.GP6, J4.3 (Pin_3); no longer U1.GP7
- net IN_2_4: now also U1.GP8, J13.2 (Pin_2); no longer U1.GP10
- net PWR_IN: now also J15.1 (Pin_1)
- net RST: now also J3.6 (Pin_6); no longer J2.4 (Pin_4)
- net SCL: now also J3.5 (Pin_5); no longer J3.3 (Pin_3)
- net SDA: now also J3.4 (Pin_4); no longer J3.2 (Pin_2)
- net TOGG_ACT_1: now also J14.2 (Pin_2)
- net TOGG_ACT_2: now also J14.1 (Pin_1)
- net at Q1.2 (G), SW2.3 (A): now also R1.1
- net LED_PIN_1 renamed GP13
- net GP13: now also J1.3 (Pin_3)
- net LED_PIN_2 renamed GP14
- net GP14: now also J1.2 (Pin_2)
- net LED_PIN_3 renamed GP15
- net GP15: now also J1.1 (Pin_1)
